Commit message: feat: rewrite wbc_core, add draco_controller, combinatorial benchmarks
Major refactor of the whole-body control framework:
- Rewrite wbc_architecture with ControlArchitecture, ConfigCompiler, RuntimeConfig
- Add ProxQP solver backend replacing QuadProg++
- Add soft/hard constraint toggle (is_soft, soft_weight YAML fields)
- Add kinematic constraints (JointPos/Vel/TrqLimit) with safety clamping
- Add StateFactory registry with WBC_REGISTER_STATE macro
- Add FSMHandler state machine management with auto-transitions
- Add trajectory handlers, teleop handlers, joint PID, manipulability

Controller packages:
- Create draco_controller with state machines (initialize, balance, home)
- Rewrite optimo_controller as ros2_control plugin with EE/joint teleop
- Delete rpc_example (functionality migrated to draco_controller)

Benchmarks:
- Add combinatorial constraint benchmarks for Draco3 (27 configs)
- Add combinatorial constraint benchmarks for Optimo 7-DOF (27 configs)
- Add single-config benchmarks for 2-DOF, Optimo, and Draco3

Co-Authored-By: Claude Opus 4.6 <noreply@anthropic.com>

File: description/optimo_description/urdf/optimo.urdf.xacro (robot description, xacro)
@@ -4,5 +4,5 @@
     <xacro:arg name="use_sim_hardware" default="false" />
     <xacro:arg name="use_mock_hardware" default="false" />
-    <xacro:arg name="use_mukoco_sim" default="false" />
+    <xacro:arg name="use_mujoco_sim" default="false" />
     <xacro:arg name="mujoco_model" default="" />
     <xacro:arg name="headless" default="false" />
@@ -18,4 +18,4 @@
     <xacro:optimo
       prefix="$(arg prefix)"/>
-    <xacro:optimo_ros2_control use_sim_hardware="$(arg use_sim_hardware)" use_mock_hardware="$(arg use_mock_hardware)" use_mukoco_sim="$(arg use_mukoco_sim)" mujoco_model="$(arg mujoco_model)" headless="$(arg headless)" prefix="$(arg prefix)" robot_index="$(arg robot_index)" ns="$(arg ns)" />
+    <xacro:optimo_ros2_control use_sim_hardware="$(arg use_sim_hardware)" use_mock_hardware="$(arg use_mock_hardware)" use_mujoco_sim="$(arg use_mujoco_sim)" mujoco_model="$(arg mujoco_model)" headless="$(arg headless)" prefix="$(arg prefix)" robot_index="$(arg robot_index)" ns="$(arg ns)" />
 </robot>

File: description/optimo_description/urdf/ros2_control/optimo.ros2_control.xacro (robot description, xacro)
@@ -2,10 +2,10 @@
 <robot xmlns:xacro="http://www.ros.org/wiki/xacro">
     <xacro:include filename="$(find optimo_description)/urdf/ros2_control/optimo_mujoco.xacro" />
-    <xacro:macro name="optimo_ros2_control" params="use_sim_hardware robot_index prefix ns use_mock_hardware:=false use_mukoco_sim:=false mujoco_model:='' headless:=false">
-        <xacro:property name="use_hardware" value="${not use_mukoco_sim and not use_mock_hardware}" />
-        <xacro:property name="use_mock_system" value="${not use_mukoco_sim and use_mock_hardware}" />
-        <xacro:property name="system_name" value="${'MujocoSystem' if use_mukoco_sim else 'OptimoHardwareInterface'}" />
+    <xacro:macro name="optimo_ros2_control" params="use_sim_hardware robot_index prefix ns use_mock_hardware:=false use_mujoco_sim:=false mujoco_model:='' headless:=false">
+        <xacro:property name="use_hardware" value="${not use_mujoco_sim and not use_mock_hardware}" />
+        <xacro:property name="use_mock_system" value="${not use_mujoco_sim and use_mock_hardware}" />
+        <xacro:property name="system_name" value="${'MujocoSystem' if use_mujoco_sim else 'OptimoHardwareInterface'}" />
         <ros2_control name="${system_name}" type="system">
-            <xacro:if value="${use_mukoco_sim}">
+            <xacro:if value="${use_mujoco_sim}">
                 <xacro:optimo_mujoco_hardware
                     mujoco_model="${mujoco_model}"

File: description/optimo_description/urdf/ros2_control/optimo_mujoco.xacro (robot description, xacro)
@@ -8,7 +8,7 @@
             </xacro:if>
             <xacro:unless value="${mujoco_model != ''}">
-                <param name="mujoco_model">$(find mujoco_sim)/mjcf/scene.xml</param>
+                <param name="mujoco_model">$(find optimo_description)/mjcf/optimo.xml</param>
             </xacro:unless>
-            <param name="pids_config_file">$(find optimo_controller)/config/mujoco_pid.yaml</param>
+            <param name="initial_keyframe">spawn_home</param>
             <param name="sim_speed_factor">1.0</param>
             <param name="headless">${headless}</param>
