Commit message: wip

File: description/optimo_description/urdf/optimo.urdf (robot description, URDF)
Before this commit: robot optimo, 12 links, 11 joints
Links:
- removed link base_link
- removed link end_effector
- removed link link0
- removed link link1
- removed link link2
- removed link link3
- removed link link4
- removed link link5
- removed link link6
- removed link link7
- removed link stand
- added link optimo_base_link
- added link optimo_end_effector
- added link optimo_link0, mass 1; collision mesh filename=meshes/col0.stl; visual mesh filename=meshes/link0.stl
- added link optimo_link1, mass 4.152; collision mesh filename=meshes/col1.stl; visual mesh filename=meshes/link1.stl
- added link optimo_link2, mass 1.72; collision mesh filename=meshes/col2.stl; visual mesh filename=meshes/link2.stl
- added link optimo_link3, mass 4.310; collision mesh filename=meshes/col3.stl; visual mesh filename=meshes/link3.stl
- added link optimo_link4, mass 1.09; collision mesh filename=meshes/col4.stl; visual mesh filename=meshes/link4.stl
- added link optimo_link5, mass 2.23; collision mesh filename=meshes/col5.stl; visual mesh filename=meshes/link5.stl
- added link optimo_link6, mass 1.138; collision mesh filename=meshes/col6.stl; visual mesh filename=meshes/link6.stl
- added link optimo_link7, mass .88; collision mesh filename=meshes/col7.stl; visual mesh filename=meshes/link7.stl
- added link optimo_stand; collision box size=0.5 0.5 1; visual box size=0.5 0.5 1
Joints:
- removed joint base_link_to_link0
- removed joint ee_joint
- removed joint joint1
- removed joint joint2
- removed joint joint3
- removed joint joint4
- removed joint joint5
- removed joint joint6
- removed joint joint7
- removed joint stand_to_base_link
- removed joint world_to_stand
- added joint optimo_base_link_to_link0: type fixed, parent optimo_base_link, child optimo_link0, origin xyz=0 0 .27 rpy=0 0 0
- added joint optimo_ee_joint: type fixed, parent optimo_link7, child optimo_end_effector, origin xyz=0 0 0.15 rpy=0 0 0
- added joint optimo_joint1: type revolute, parent optimo_link0, child optimo_link1, origin xyz=0 0 0 rpy=0 0 0, axis 0 0 1, limit lower=-2.0943951012 upper=2.0943951012 effort=79 velocity=10
- added joint optimo_joint2: type revolute, parent optimo_link1, child optimo_link2, origin xyz=0 0 0 rpy=1.5707963267948966 0 0, axis 0 0 1, limit lower=1.0471975506 upper=3.8397243521999997 effort=95 velocity=10
- added joint optimo_joint3: type revolute, parent optimo_link2, child optimo_link3, origin xyz=0 -0.4 0 rpy=1.5707963267948966 0 0, axis 0 0 1, limit lower=-2.0943951012 upper=2.0943951012 effort=32 velocity=10
- added joint optimo_joint4: type revolute, parent optimo_link3, child optimo_link4, origin xyz=0 0 0 rpy=-1.5707963267948966 0 0, axis 0 0 1, limit lower=-2.53072741395 upper=2.53072741395 effort=40 velocity=10
- added joint optimo_joint5: type revolute, parent optimo_link4, child optimo_link5, origin xyz=0 -0.4 0 rpy=1.5707963267948966 0 0, axis 0 0 1, limit lower=-2.6179938765 upper=2.6179938765 effort=15 velocity=10
- added joint optimo_joint6: type revolute, parent optimo_link5, child optimo_link6, origin xyz=0 0 0 rpy=-1.5707963267948966 0 0, axis 0 0 1, limit lower=-2.0943951012 upper=2.0943951012 effort=15 velocity=10
- added joint optimo_joint7: type revolute, parent optimo_link6, child optimo_link7, origin xyz=0 0 0 rpy=1.5707963267948966 0 0, axis 0 0 1, limit lower=-2.0943951012 upper=2.0943951012 effort=15 velocity=10
- added joint optimo_stand_to_base_link: type fixed, parent optimo_stand, child optimo_base_link, origin xyz=0 0 0 rpy=0 0 0
- added joint optimo_world_to_stand: type fixed, parent world, child optimo_stand, origin xyz=0 0 0 rpy=0 0 0

File: description/optimo_description/urdf/optimo.urdf.xacro (robot description, xacro)
@@ -7,15 +7,13 @@
     <xacro:arg name="mujoco_model" default="" />
     <xacro:arg name="headless" default="false" />
-    <xacro:arg name="prefix" default=""/>
     <xacro:arg name="robot_index" default="0"/>
     <xacro:arg name="ns" default="optimo"/>
     <!-- Import files -->
-    <xacro:include filename="$(find optimo_description)/urdf/xacro/optimo.common.xacro" />
-    <xacro:include filename="$(find optimo_description)/urdf/xacro/optimo.xacro" />
-    <xacro:include filename="$(find optimo_description)/urdf/ros2_control/optimo.ros2_control.xacro" />
+    <xacro:include filename="xacro/optimo.common.xacro" />
+    <xacro:include filename="xacro/optimo.xacro" />
+    <xacro:include filename="ros2_control/optimo.ros2_control.xacro" />
     <link name="world"/>
     <!-- Actually add the arm, and ros2 control -->
-    <xacro:optimo
-      prefix="$(arg prefix)"/>
-    <xacro:optimo_ros2_control use_sim_hardware="$(arg use_sim_hardware)" use_mock_hardware="$(arg use_mock_hardware)" use_mujoco_sim="$(arg use_mujoco_sim)" mujoco_model="$(arg mujoco_model)" headless="$(arg headless)" prefix="$(arg prefix)" robot_index="$(arg robot_index)" ns="$(arg ns)" />
+    <xacro:optimo/>
+    <xacro:optimo_ros2_control use_sim_hardware="$(arg use_sim_hardware)" use_mock_hardware="$(arg use_mock_hardware)" use_mujoco_sim="$(arg use_mujoco_sim)" mujoco_model="$(arg mujoco_model)" headless="$(arg headless)" robot_index="$(arg robot_index)" ns="$(arg ns)" />
 </robot>

File: description/optimo_description/urdf/ros2_control/optimo.ros2_control.xacro (robot description, xacro)
@@ -1,6 +1,6 @@
 <?xml version="1.0"?>
 <robot xmlns:xacro="http://www.ros.org/wiki/xacro">
-    <xacro:include filename="$(find optimo_description)/urdf/ros2_control/optimo_mujoco.xacro" />
-    <xacro:macro name="optimo_ros2_control" params="use_sim_hardware robot_index prefix ns use_mock_hardware:=false use_mujoco_sim:=false mujoco_model:='' headless:=false">
+    <xacro:include filename="optimo_mujoco.xacro" />
+    <xacro:macro name="optimo_ros2_control" params="use_sim_hardware robot_index ns use_mock_hardware:=false use_mujoco_sim:=false mujoco_model:='' headless:=false">
         <xacro:property name="use_hardware" value="${not use_mujoco_sim and not use_mock_hardware}" />
         <xacro:property name="use_mock_system" value="${not use_mujoco_sim and use_mock_hardware}" />
@@ -12,5 +12,16 @@
                     headless="${headless}" />
             </xacro:if>
-            <joint name="${prefix}joint1">
+            <joint name="optimo_joint1">
+                <command_interface name="position" />
+                <command_interface name="velocity" />
+                <command_interface name="effort">
+                    <param name="min">-79</param>
+                    <param name="max">79</param>
+                </command_interface>
+                <state_interface name="position" />
+                <state_interface name="velocity" />
+                <state_interface name="effort" />
+            </joint>
+            <joint name="optimo_joint2">
                 <command_interface name="position" />
                 <command_interface name="velocity" />
@@ -23,10 +34,10 @@
                 <state_interface name="effort" />
             </joint>
-            <joint name="${prefix}joint2">
+            <joint name="optimo_joint3">
                 <command_interface name="position" />
                 <command_interface name="velocity" />
                 <command_interface name="effort">
-                    <param name="min">-95</param>
-                    <param name="max">95</param>
+                    <param name="min">-32</param>
+                    <param name="max">32</param>
                 </command_interface>
                 <state_interface name="position" />
@@ -34,5 +45,5 @@
                 <state_interface name="effort" />
             </joint>
-            <joint name="${prefix}joint3">
+            <joint name="optimo_joint4">
                 <command_interface name="position" />
                 <command_interface name="velocity" />
@@ -45,16 +56,5 @@
                 <state_interface name="effort" />
             </joint>
-            <joint name="${prefix}joint4">
-                <command_interface name="position" />
-                <command_interface name="velocity" />
-                <command_interface name="effort">
-                    <param name="min">-40</param>
-                    <param name="max">40</param>
-                </command_interface>
-                <state_interface name="position" />
-                <state_interface name="velocity" />
-                <state_interface name="effort" />
-            </joint>
-            <joint name="${prefix}joint5">
+            <joint name="optimo_joint5">
                 <command_interface name="position" />
                 <command_interface name="velocity" />
@@ -67,5 +67,5 @@
                 <state_interface name="effort" />
             </joint>
-            <joint name="${prefix}joint6">
+            <joint name="optimo_joint6">
                 <command_interface name="position" />
                 <command_interface name="velocity" />
@@ -78,5 +78,5 @@
                 <state_interface name="effort" />
             </joint>
-            <joint name="${prefix}joint7">
+            <joint name="optimo_joint7">
                 <command_interface name="position" />
                 <command_interface name="velocity" />

File: description/optimo_description/urdf/ros2_control/optimo_mujoco.xacro (robot description, xacro)
@@ -10,5 +10,4 @@
                 <param name="mujoco_model">$(find optimo_description)/mjcf/optimo.xml</param>
             </xacro:unless>
-            <param name="pids_config_file">$(find optimo_description)/config/mujoco_pid_gains.yaml</param>
             <param name="initial_keyframe">spawn_home</param>
             <param name="sim_speed_factor">1.0</param>
