Commit message: wip

File: description/plato_description/urdf/plato.urdf.xacro (robot description, xacro)
@@ -4,12 +4,19 @@
     <xacro:arg name="use_aristo_hand" default="false" />
     <xacro:arg name="use_sim_hardware" default="false" />
+    <xacro:arg name="use_mujoco_sim" default="false" />
+    <xacro:arg name="mujoco_model" default="" />
+    <xacro:arg name="headless" default="false" />
     <xacro:arg name="prefix" default=""/>
     <xacro:arg name="robot_index" default="0"/>
-    <xacro:arg name="ns" default="optimo"/>
+    <xacro:arg name="ns" default="plato"/>
     <!-- Import files -->
     <xacro:include filename="$(find plato_description)/urdf/xacro/optimo.common.xacro" />
     <xacro:include filename="$(find plato_description)/urdf/xacro/optimo.xacro" />
+    <xacro:include filename="$(find plato_description)/urdf/xacro/aristo_description.xacro" />
     <xacro:include filename="$(find plato_description)/urdf/ros2_control/optimo.ros2_control.xacro" />
-    <xacro:include filename="$(find plato_description)/urdf/xacro/aristo_description.xacro" />
+    <xacro:include filename="$(find plato_description)/urdf/ros2_control/plato_mujoco.xacro" />
+    <mujoco>
+      <compiler meshdir="meshes/"/>
+    </mujoco>
     <link name="world"/>
     <!-- Add the arm, optional hand, and ros2_control -->
@@ -25,4 +32,182 @@
       </joint>
     </xacro:if>
-    <xacro:optimo_ros2_control use_sim_hardware="$(arg use_sim_hardware)" prefix="$(arg prefix)" robot_index="$(arg robot_index)" ns="$(arg ns)" />
+    <!-- MuJoCo sim: unified ros2_control with all 15 joints -->
+    <xacro:if value="$(arg use_mujoco_sim)">
+      <ros2_control name="MujocoSystem" type="system">
+        <xacro:plato_mujoco_hardware
+            mujoco_model="$(arg mujoco_model)"
+            headless="$(arg headless)" />
+        <!-- Arm joints (7-DOF) -->
+        <joint name="joint1">
+            <command_interface name="position" />
+            <command_interface name="velocity" />
+            <command_interface name="effort">
+                <param name="min">-79</param>
+                <param name="max">79</param>
+            </command_interface>
+            <state_interface name="position" />
+            <state_interface name="velocity" />
+            <state_interface name="effort" />
+        </joint>
+        <joint name="joint2">
+            <command_interface name="position" />
+            <command_interface name="velocity" />
+            <command_interface name="effort">
+                <param name="min">-95</param>
+                <param name="max">95</param>
+            </command_interface>
+            <state_interface name="position" />
+            <state_interface name="velocity" />
+            <state_interface name="effort" />
+        </joint>
+        <joint name="joint3">
+            <command_interface name="position" />
+            <command_interface name="velocity" />
+            <command_interface name="effort">
+                <param name="min">-32</param>
+                <param name="max">32</param>
+            </command_interface>
+            <state_interface name="position" />
+            <state_interface name="velocity" />
+            <state_interface name="effort" />
+        </joint>
+        <joint name="joint4">
+            <command_interface name="position" />
+            <command_interface name="velocity" />
+            <command_interface name="effort">
+                <param name="min">-40</param>
+                <param name="max">40</param>
+            </command_interface>
+            <state_interface name="position" />
+            <state_interface name="velocity" />
+            <state_interface name="effort" />
+        </joint>
+        <joint name="joint5">
+            <command_interface name="position" />
+            <command_interface name="velocity" />
+            <command_interface name="effort">
+                <param name="min">-15</param>
+                <param name="max">15</param>
+            </command_interface>
+            <state_interface name="position" />
+            <state_interface name="velocity" />
+            <state_interface name="effort" />
+        </joint>
+        <joint name="joint6">
+            <command_interface name="position" />
+            <command_interface name="velocity" />
+            <command_interface name="effort">
+                <param name="min">-15</param>
+                <param name="max">15</param>
+            </command_interface>
+            <state_interface name="position" />
+            <state_interface name="velocity" />
+            <state_interface name="effort" />
+        </joint>
+        <joint name="joint7">
+            <command_interface name="position" />
+            <command_interface name="velocity" />
+            <command_interface name="effort">
+                <param name="min">-15</param>
+                <param name="max">15</param>
+            </command_interface>
+            <state_interface name="position" />
+            <state_interface name="velocity" />
+            <state_interface name="effort" />
+        </joint>
+        <!-- Hand joints (8-DOF) -->
+        <joint name="aristo_joint1">
+            <command_interface name="position" />
+            <command_interface name="velocity" />
+            <command_interface name="effort">
+                <param name="min">-10</param>
+                <param name="max">10</param>
+            </command_interface>
+            <state_interface name="position" />
+            <state_interface name="velocity" />
+            <state_interface name="effort" />
+        </joint>
+        <joint name="aristo_joint2">
+            <command_interface name="position" />
+            <command_interface name="velocity" />
+            <command_interface name="effort">
+                <param name="min">-10</param>
+                <param name="max">10</param>
+            </command_interface>
+            <state_interface name="position" />
+            <state_interface name="velocity" />
+            <state_interface name="effort" />
+        </joint>
+        <joint name="aristo_joint3">
+            <command_interface name="position" />
+            <command_interface name="velocity" />
+            <command_interface name="effort">
+                <param name="min">-10</param>
+                <param name="max">10</param>
+            </command_interface>
+            <state_interface name="position" />
+            <state_interface name="velocity" />
+            <state_interface name="effort" />
+        </joint>
+        <joint name="aristo_joint4">
+            <command_interface name="position" />
+            <command_interface name="velocity" />
+            <command_interface name="effort">
+                <param name="min">-10</param>
+                <param name="max">10</param>
+            </command_interface>
+            <state_interface name="position" />
+            <state_interface name="velocity" />
+            <state_interface name="effort" />
+        </joint>
+        <joint name="aristo_joint5">
+            <command_interface name="position" />
+            <command_interface name="velocity" />
+            <command_interface name="effort">
+                <param name="min">-10</param>
+                <param name="max">10</param>
+            </command_interface>
+            <state_interface name="position" />
+            <state_interface name="velocity" />
+            <state_interface name="effort" />
+        </joint>
+        <joint name="aristo_joint6">
+            <command_interface name="position" />
+            <command_interface name="velocity" />
+            <command_interface name="effort">
+                <param name="min">-10</param>
+                <param name="max">10</param>
+            </command_interface>
+            <state_interface name="position" />
+            <state_interface name="velocity" />
+            <state_interface name="effort" />
+        </joint>
+        <joint name="aristo_joint7">
+            <command_interface name="position" />
+            <command_interface name="velocity" />
+            <command_interface name="effort">
+                <param name="min">-10</param>
+                <param name="max">10</param>
+            </command_interface>
+            <state_interface name="position" />
+            <state_interface name="velocity" />
+            <state_interface name="effort" />
+        </joint>
+        <joint name="aristo_joint8">
+            <command_interface name="position" />
+            <command_interface name="velocity" />
+            <command_interface name="effort">
+                <param name="min">-10</param>
+                <param name="max">10</param>
+            </command_interface>
+            <state_interface name="position" />
+            <state_interface name="velocity" />
+            <state_interface name="effort" />
+        </joint>
+      </ros2_control>
+    </xacro:if>
+    <!-- Non-MuJoCo: use original Ignition/hardware ros2_control (arm only) -->
+    <xacro:unless value="$(arg use_mujoco_sim)">
+      <xacro:optimo_ros2_control use_sim_hardware="$(arg use_sim_hardware)" prefix="$(arg prefix)" robot_index="$(arg robot_index)" ns="$(arg ns)" />
+    </xacro:unless>
 </robot>

File: description/plato_description/urdf/xacro/aristo_description.xacro (robot description, xacro)
@@ -26,5 +26,5 @@
         <origin xyz="1.14624e-05 -0.0735402 0.00270001" rpy="0 0 0"/>
         <geometry>
-          <mesh filename="package://plato_description/meshes/hand_base.stl"/>
+          <mesh filename="package://plato_description/urdf/meshes/hand_base.stl"/>
         </geometry>
         <material name="hand_base_parts_material">
@@ -35,5 +35,5 @@
         <origin xyz="1.14624e-05 -0.0735402 0.00270001" rpy="0 0 0"/>
         <geometry>
-          <mesh filename="package://plato_description/meshes/hand_base.stl"/>
+          <mesh filename="package://plato_description/urdf/meshes/col_hand_base.stl"/>
         </geometry>
       </collision>
@@ -66,5 +66,5 @@
         <origin xyz="5.08388e-05 -0.0186588 0.0228524" rpy="-1.5708 0 -2.97318e-15"/>
         <geometry>
-          <mesh filename="package://plato_description/meshes/thumb_metacarpal.stl"/>
+          <mesh filename="package://plato_description/urdf/meshes/thumb_metacarpal.stl"/>
         </geometry>
         <material name="thumb_metacarpal_parts_material">
@@ -75,5 +75,5 @@
         <origin xyz="5.08388e-05 -0.0186588 0.0228524" rpy="-1.5708 0 -2.97318e-15"/>
         <geometry>
-          <mesh filename="package://plato_description/meshes/thumb_metacarpal.stl"/>
+          <mesh filename="package://plato_description/urdf/meshes/col_thumb_metacarpal.stl"/>
         </geometry>
       </collision>
@@ -89,5 +89,5 @@
         <origin xyz="0.00119788 -0.0189545 -0.0225138" rpy="0 0 -1.5708"/>
         <geometry>
-          <mesh filename="package://plato_description/meshes/thumb_actuators.stl"/>
+          <mesh filename="package://plato_description/urdf/meshes/thumb_actuators.stl"/>
         </geometry>
         <material name="thumb_actuators_parts_material">
@@ -98,5 +98,5 @@
         <origin xyz="0.00119788 -0.0189545 -0.0225138" rpy="0 0 -1.5708"/>
         <geometry>
-          <mesh filename="package://plato_description/meshes/thumb_actuators.stl"/>
+          <mesh filename="package://plato_description/urdf/meshes/col_thumb_actuators.stl"/>
         </geometry>
       </collision>
@@ -112,5 +112,5 @@
         <origin xyz="0.0275353 8.61887e-05 0.00673205" rpy="1.5708 -1.5708 0"/>
         <geometry>
-          <mesh filename="package://plato_description/meshes/thumb_proximal.stl"/>
+          <mesh filename="package://plato_description/urdf/meshes/thumb_proximal.stl"/>
         </geometry>
         <material name="thumb_proximal_parts_material">
@@ -121,5 +121,5 @@
         <origin xyz="0.0275353 8.61887e-05 0.00673205" rpy="1.5708 -1.5708 0"/>
         <geometry>
-          <mesh filename="package://plato_description/meshes/thumb_proximal.stl"/>
+          <mesh filename="package://plato_description/urdf/meshes/col_thumb_proximal.stl"/>
         </geometry>
       </collision>
@@ -135,5 +135,5 @@
         <origin xyz="-0.0330685 -0.00101822 -0.00300906" rpy="-1.5708 -1.5708 0"/>
         <geometry>
-          <mesh filename="package://plato_description/meshes/thumb_distal.stl"/>
+          <mesh filename="package://plato_description/urdf/meshes/thumb_distal.stl"/>
         </geometry>
         <material name="thumb_distal_parts_material">
@@ -144,5 +144,5 @@
         <origin xyz="-0.0330685 -0.00101822 -0.00300906" rpy="-1.5708 -1.5708 0"/>
         <geometry>
-          <mesh filename="package://plato_description/meshes/thumb_distal.stl"/>
+          <mesh filename="package://plato_description/urdf/meshes/col_thumb_distal.stl"/>
         </geometry>
       </collision>
@@ -187,5 +187,5 @@
         <origin xyz="0.0275353 -8.61566e-05 0.00673211" rpy="1.5708 -1.5708 0"/>
         <geometry>
-          <mesh filename="package://plato_description/meshes/index_proximal.stl"/>
+          <mesh filename="package://plato_description/urdf/meshes/index_proximal.stl"/>
         </geometry>
         <material name="index_proximal_parts_material">
@@ -196,5 +196,5 @@
         <origin xyz="0.0275353 -8.61566e-05 0.00673211" rpy="1.5708 -1.5708 0"/>
         <geometry>
-          <mesh filename="package://plato_description/meshes/index_proximal.stl"/>
+          <mesh filename="package://plato_description/urdf/meshes/col_index_proximal.stl"/>
         </geometry>
       </collision>
@@ -210,5 +210,5 @@
         <origin xyz="-0.0330685 0.00101822 -0.00299094" rpy="-1.5708 -1.5708 0"/>
         <geometry>
-          <mesh filename="package://plato_description/meshes/index_distal.stl"/>
+          <mesh filename="package://plato_description/urdf/meshes/index_distal.stl"/>
         </geometry>
         <material name="index_distal_parts_material">
@@ -219,5 +219,5 @@
         <origin xyz="-0.0330685 0.00101822 -0.00299094" rpy="-1.5708 -1.5708 0"/>
         <geometry>
-          <mesh filename="package://plato_description/meshes/index_distal.stl"/>
+          <mesh filename="package://plato_description/urdf/meshes/col_index_distal.stl"/>
         </geometry>
       </collision>
@@ -279,5 +279,5 @@
         <origin xyz="0.0275353 -8.61887e-05 -0.00673205" rpy="1.5708 -1.5708 0"/>
         <geometry>
-          <mesh filename="package://plato_description/meshes/middle_proximal.stl"/>
+          <mesh filename="package://plato_description/urdf/meshes/middle_proximal.stl"/>
         </geometry>
         <material name="middle_proximal_parts_material">
@@ -288,5 +288,5 @@
         <origin xyz="0.0275353 -8.61887e-05 -0.00673205" rpy="1.5708 -1.5708 0"/>
         <geometry>
-          <mesh filename="package://plato_description/meshes/middle_proximal.stl"/>
+          <mesh filename="package://plato_description/urdf/meshes/col_middle_proximal.stl"/>
         </geometry>
       </collision>
@@ -302,5 +302,5 @@
         <origin xyz="-0.0330685 0.00101822 0.00300906" rpy="-1.5708 -1.5708 0"/>
         <geometry>
-          <mesh filename="package://plato_description/meshes/middle_distal.stl"/>
+          <mesh filename="package://plato_description/urdf/meshes/middle_distal.stl"/>
         </geometry>
         <material name="middle_distal_parts_material">
@@ -311,5 +311,5 @@
         <origin xyz="-0.0330685 0.00101822 0.00300906" rpy="-1.5708 -1.5708 0"/>
         <geometry>
-          <mesh filename="package://plato_description/meshes/middle_distal.stl"/>
+          <mesh filename="package://plato_description/urdf/meshes/col_middle_distal.stl"/>
         </geometry>
       </collision>
