Commit message: wip

File: description/plato_description/urdf/xacro/optimo.xacro (robot description, xacro)
@@ -1,85 +1,66 @@
 <?xml version="1.0"?>
 <robot xmlns:xacro="http://www.ros.org/wiki/xacro">
-    <xacro:macro name="optimo" params="prefix:='' standalone:=true">
-        <!-- Default joint limits (upright) -->
+    <xacro:macro name="optimo" params="prefix:=''">
+        <!-- Joint limits (from hardware safety config) -->
         <xacro:property name="joint1_lower" value="${DtR*-120}" />
         <xacro:property name="joint1_upper" value="${DtR*120}" />
-        <xacro:property name="joint2_lower" value="${DtR*65}" />
-        <xacro:property name="joint2_upper" value="${DtR*195}" />
+        <xacro:property name="joint2_lower" value="${DtR*60}" />
+        <xacro:property name="joint2_upper" value="${DtR*220}" />
         <xacro:property name="joint3_lower" value="${DtR*-120}" />
         <xacro:property name="joint3_upper" value="${DtR*120}" />
-        <xacro:property name="joint4_lower" value="${DtR*-140}" />
-        <xacro:property name="joint4_upper" value="${DtR*5}" />
+        <xacro:property name="joint4_lower" value="${DtR*-145}" />
+        <xacro:property name="joint4_upper" value="${DtR*145}" />
         <xacro:property name="joint5_lower" value="${DtR*-150}" />
         <xacro:property name="joint5_upper" value="${DtR*150}" />
-        <xacro:property name="joint6_lower" value="${DtR*-115}" />
-        <xacro:property name="joint6_upper" value="${DtR*115}" />
+        <xacro:property name="joint6_lower" value="${DtR*-120}" />
+        <xacro:property name="joint6_upper" value="${DtR*120}" />
         <xacro:property name="joint7_lower" value="${DtR*-120}" />
         <xacro:property name="joint7_upper" value="${DtR*120}" />
-        <!-- Joint limit properties -->
-        <xacro:if value="${prefix == 'left_arm_'}">
-            <!-- Left arm joint limits -->
-            <xacro:property name="joint1_lower" value="${DtR*-120}" />
-            <xacro:property name="joint1_upper" value="${DtR*60}" />
-            <xacro:property name="joint2_lower" value="${DtR*190}" />
-            <xacro:property name="joint2_upper" value="${DtR*280}" />
-            <xacro:property name="joint3_lower" value="${DtR*-210}" />
-            <xacro:property name="joint3_upper" value="${DtR*30}" />
-            <xacro:property name="joint4_lower" value="${DtR*-5}" />
-            <xacro:property name="joint4_upper" value="${DtR*140}" />
-        </xacro:if>
-        <xacro:if value="${prefix == 'right_arm_'}">
-            <!-- Right arm joint limits -->
-            <xacro:property name="joint1_lower" value="${DtR*-60}" />
-            <xacro:property name="joint1_upper" value="${DtR*120}" />
-            <xacro:property name="joint2_lower" value="${DtR*80}" />
-            <xacro:property name="joint2_upper" value="${DtR*170}" />
-            <xacro:property name="joint3_lower" value="${DtR*-30}" />
-            <xacro:property name="joint3_upper" value="${DtR*210}" />
-            <xacro:property name="joint4_lower" value="${DtR*-140}" />
-            <xacro:property name="joint4_upper" value="${DtR*5}" />
-        </xacro:if>
-        <!-- If standalone, connect world link and mounting stand to the base of the arm.-->
-        <xacro:if value="${standalone}">
-            <joint name="${prefix}world_to_stand" type="fixed">
-                <parent link="world" />
-                <child link="${prefix}stand" />
-                <origin xyz="0 0 1" rpy="0 0 -1.57" />
-            </joint>
-            <link name="${prefix}stand">
-                <visual>
-                    <origin xyz="0 0 -0.5" rpy="0 0 0" />
-                    <geometry>
-                        <box size="0.3 0.3 1" />
-                    </geometry>
-                    <material name="white" />
-                </visual>
-                <collision>
-                    <origin xyz="0 0 -0.5" rpy="0 0 0" />
-                    <geometry>
-                        <box size="0.3 0.3 1" />
-                    </geometry>
-                </collision>
-            </link>
-            <joint name="${prefix}stand_to_link0" type="fixed">
-                <parent link="${prefix}stand" />
-                <child link="${prefix}link0" />
-                <origin xyz="0 0 0" rpy="0 0 0" />
-            </joint>
-        </xacro:if>
+        <!-- Stand: connects world to base_link -->
+        <joint name="${prefix}world_to_stand" type="fixed">
+            <parent link="world" />
+            <child link="${prefix}stand" />
+            <origin xyz="0 0 0" rpy="0 0 0" />
+        </joint>
+        <link name="${prefix}stand">
+            <visual>
+                <origin xyz="0 0 -0.5" rpy="0 0 0" />
+                <geometry>
+                    <box size="0.5 0.5 1" />
+                </geometry>
+                <material name="white" />
+            </visual>
+            <collision>
+                <origin xyz="0 0 -0.5" rpy="0 0 0" />
+                <geometry>
+                    <box size="0.5 0.5 1" />
+                </geometry>
+            </collision>
+        </link>
+        <joint name="${prefix}stand_to_base_link" type="fixed">
+            <parent link="${prefix}stand" />
+            <child link="${prefix}base_link" />
+            <origin xyz="0 0 0" rpy="0 0 0" />
+        </joint>
+        <link name="${prefix}base_link"/>
+        <joint name="${prefix}base_link_to_link0" type="fixed">
+            <parent link="${prefix}base_link" />
+            <child link="${prefix}link0" />
+            <origin xyz="0 0 .27" rpy="0 0 0" />
+        </joint>
         <!-- Base Link -->
         <link name="${prefix}link0">
             <visual>
                 <geometry>
-                    <mesh filename="package://plato_description/meshes/link0.stl" />
-                </geometry>
-                <material name="blue" />
-            </visual>
-            <collision>
-                <geometry>
-                    <mesh filename="package://plato_description/meshes/col0.stl" />
-                </geometry>
-            </collision>
-            <inertial>                <!-- Doesn't matter, just placeholder values -->
+                    <mesh filename="package://plato_description/urdf/meshes/link0.stl" />
+                </geometry>
+                <material name="blue" />
+            </visual>
+            <collision>
+                <geometry>
+                    <mesh filename="package://plato_description/urdf/meshes/col0.stl" />
+                </geometry>
+            </collision>
+            <inertial>
                 <origin xyz="0 0 0" />
                 <mass value="1" />
@@ -99,16 +80,14 @@
                 <origin xyz="0 0 0" rpy="${PI/2} 0 0" />
                 <geometry>
-                    <mesh filename="package://plato_description/meshes/link1.stl" />
-                </geometry>
-                <material name="white" />
-            </visual>
-            <collision>
-                <origin xyz="0 0 0" rpy="${PI/2} 0 0" />
-                <geometry>
-                    <mesh filename="package://plato_description/meshes/col1.stl" />
-                </geometry>
-            </collision>
-            <!-- Inertia values could be taken from yaml, but do not seem realistic so some estimations
-        were made instead...-->
+                    <mesh filename="package://plato_description/urdf/meshes/link1.stl" />
+                </geometry>
+                <material name="white" />
+            </visual>
+            <collision>
+                <origin xyz="0 0 0" rpy="${PI/2} 0 0" />
+                <geometry>
+                    <mesh filename="package://plato_description/urdf/meshes/col1.stl" />
+                </geometry>
+            </collision>
             <inertial>
                 <origin xyz="0 -0.01549 -0.01635 " />
@@ -129,12 +108,12 @@
                 <origin xyz="0 0 0" rpy="${PI/2} 0 0" />
                 <geometry>
-                    <mesh filename="package://plato_description/meshes/link2.stl" />
-                </geometry>
-                <material name="blue" />
-            </visual>
-            <collision>
-                <origin xyz="0 0 0" rpy="${PI/2} 0 0" />
-                <geometry>
-                    <mesh filename="package://plato_description/meshes/col2.stl" />
+                    <mesh filename="package://plato_description/urdf/meshes/link2.stl" />
+                </geometry>
+                <material name="blue" />
+            </visual>
+            <collision>
+                <origin xyz="0 0 0" rpy="${PI/2} 0 0" />
+                <geometry>
+                    <mesh filename="package://plato_description/urdf/meshes/col2.stl" />
                 </geometry>
             </collision>
@@ -157,12 +136,12 @@
                 <origin xyz="0 0 0" rpy="-${PI/2} 0 0" />
                 <geometry>
-                    <mesh filename="package://plato_description/meshes/link3.stl" />
-                </geometry>
-                <material name="white" />
-            </visual>
-            <collision>
-                <origin xyz="0 0 0" rpy="-${PI/2} 0 0" />
-                <geometry>
-                    <mesh filename="package://plato_description/meshes/col3.stl" />
+                    <mesh filename="package://plato_description/urdf/meshes/link3.stl" />
+                </geometry>
+                <material name="white" />
+            </visual>
+            <collision>
+                <origin xyz="0 0 0" rpy="-${PI/2} 0 0" />
+                <geometry>
+                    <mesh filename="package://plato_description/urdf/meshes/col3.stl" />
                 </geometry>
             </collision>
@@ -185,12 +164,12 @@
                 <origin xyz="0 0 0" rpy="${PI/2} 0 0" />
                 <geometry>
-                    <mesh filename="package://plato_description/meshes/link4.stl" />
-                </geometry>
-                <material name="blue" />
-            </visual>
-            <collision>
-                <origin xyz="0 0 0" rpy="${PI/2} 0 0" />
-                <geometry>
-                    <mesh filename="package://plato_description/meshes/col4.stl" />
+                    <mesh filename="package://plato_description/urdf/meshes/link4.stl" />
+                </geometry>
+                <material name="blue" />
+            </visual>
+            <collision>
+                <origin xyz="0 0 0" rpy="${PI/2} 0 0" />
+                <geometry>
+                    <mesh filename="package://plato_description/urdf/meshes/col4.stl" />
                 </geometry>
             </collision>
@@ -213,12 +192,12 @@
                 <origin xyz="0 0 0" rpy="-${PI/2} 0 0" />
                 <geometry>
-                    <mesh filename="package://plato_description/meshes/link5.stl" />
-                </geometry>
-                <material name="white" />
-            </visual>
-            <collision>
-                <origin xyz="0 0 0" rpy="-${PI/2} 0 0" />
-                <geometry>
-                    <mesh filename="package://plato_description/meshes/col5.stl" />
+                    <mesh filename="package://plato_description/urdf/meshes/link5.stl" />
+                </geometry>
+                <material name="white" />
+            </visual>
+            <collision>
+                <origin xyz="0 0 0" rpy="-${PI/2} 0 0" />
+                <geometry>
+                    <mesh filename="package://plato_description/urdf/meshes/col5.stl" />
                 </geometry>
             </collision>
@@ -241,12 +220,12 @@
                 <origin xyz="0 0 0" rpy="${PI/2} 0 0" />
                 <geometry>
-                    <mesh filename="package://plato_description/meshes/link6.stl" />
-                </geometry>
-                <material name="blue" />
-            </visual>
-            <collision>
-                <origin xyz="0 0 0" rpy="${PI/2} 0 0" />
-                <geometry>
-                    <mesh filename="package://plato_description/meshes/col6.stl" />
+                    <mesh filename="package://plato_description/urdf/meshes/link6.stl" />
+                </geometry>
+                <material name="blue" />
+            </visual>
+            <collision>
+                <origin xyz="0 0 0" rpy="${PI/2} 0 0" />
+                <geometry>
+                    <mesh filename="package://plato_description/urdf/meshes/col6.stl" />
                 </geometry>
             </collision>
@@ -268,11 +247,11 @@
             <visual>
                 <geometry>
-                    <mesh filename="package://plato_description/meshes/link7.stl" />
-                </geometry>
-                <material name="white" />
-            </visual>
-            <collision>
-                <geometry>
-                    <mesh filename="package://plato_description/meshes/col7.stl" />
+                    <mesh filename="package://plato_description/urdf/meshes/link7.stl" />
+                </geometry>
+                <material name="white" />
+            </visual>
+            <collision>
+                <geometry>
+                    <mesh filename="package://plato_description/urdf/meshes/col7.stl" />
                 </geometry>
             </collision>
