Commit message: wip

File: description/plato_description/urdf/aristo.urdf.xacro (robot description, xacro)
@@ -1,17 +1,18 @@
 <?xml version="1.0"?>
 <robot name="aristo_hand" xmlns:xacro="http://www.ros.org/wiki/xacro">
+  <xacro:arg name="fake_hardware" default="false"/>
+  <xacro:arg name="zeroing" default="false"/>
+  <xacro:arg name="actuator_config_yaml_path" default=""/>
   <!-- Root link for TF tree -->
-  <link name="world"/>
+  <link name="base_link"/>
   <!-- Includes -->
     <xacro:include filename="$(find plato_description)/urdf/xacro/aristo_description.xacro"/>
     <xacro:include filename="$(find plato_description)/urdf/ros2_control/aristo.ros2_control.xacro"/>
   <!-- Instantiate geometry/tree and ros2_control -->
-  <xacro:aristo_description
-    prefix=""/>
-  <joint name="connector_to_hand_mount" type="fixed">
-    <origin xyz="0 0 0" rpy="0 0 0"/>
-    <parent link="world"/>
-    <child link="hand_mount"/>
-  </joint>
-  <xacro:aristo_ros2_control name="aristo_ros2_control"/>
+  <xacro:aristo_description connector_link="base_link" xyz="0 0 0" rpy="0 0 0"/>
+  <xacro:aristo_ros2_control
+    name="aristo_ros2_control"
+    fake_hardware="$(arg fake_hardware)"
+    zeroing="$(arg zeroing)"
+    actuator_config_yaml_path="$(arg actuator_config_yaml_path)"/>
 </robot>

File: description/plato_description/urdf/aristo_mock_hardware.urdf.xacro (robot description, xacro)
@@ -2,23 +2,11 @@
 <!-- Wrapper URDF that calls the aristo ros2_control macro with mock hardware enabled -->
 <robot name="aristo_hand" xmlns:xacro="http://www.ros.org/wiki/xacro">
-  <!-- Root and hand connector -->
+  <!-- Provide a base connector link expected by the included description -->
   <link name="base_link"/>
-  <link name="end_effector"/>
-  <joint name="base_link_to_end_effector" type="fixed">
-    <parent link="base_link"/>
-    <child link="end_effector"/>
-    <origin xyz="0 0 0" rpy="0 0 0"/>
-  </joint>
   <!-- Include the full robot description and the ros2_control definition -->
   <xacro:include filename="$(find plato_description)/urdf/xacro/aristo_description.xacro"/>
   <xacro:include filename="$(find plato_description)/urdf/ros2_control/aristo.ros2_control.xacro"/>
   <!-- Instantiate geometry/tree and ros2_control with mock hardware enabled -->
-  <xacro:aristo_description
-    prefix=""/>
-  <joint name="connector_to_hand_mount" type="fixed">
-    <origin xyz="0 0 0" rpy="0 1.57 1.5708"/>
-    <parent link="end_effector"/>
-    <child link="hand_mount"/>
-  </joint>
+  <xacro:aristo_description connector_link="base_link" xyz="0 0 0" rpy="0 0 0"/>
   <xacro:aristo_ros2_control name="aristo_mock" fake_hardware="true"/>
 </robot>

File: description/plato_description/urdf/plato.urdf.xacro (robot description, xacro)
@@ -1,213 +1,12 @@
 <?xml version="1.0"?>
-<!-- Full URDF for Plato (Optimo arm + optional Aristo hand), including controls -->
-<robot xmlns:xacro="http://www.ros.org/wiki/xacro" name="plato">
-    <xacro:arg name="use_aristo_hand" default="false" />
-    <xacro:arg name="use_sim_hardware" default="false" />
-    <xacro:arg name="use_mujoco_sim" default="false" />
-    <xacro:arg name="mujoco_model" default="" />
-    <xacro:arg name="headless" default="false" />
-    <xacro:arg name="prefix" default=""/>
-    <xacro:arg name="robot_index" default="0"/>
-    <xacro:arg name="ns" default="plato"/>
-    <!-- Import files -->
-    <xacro:include filename="$(find plato_description)/urdf/xacro/optimo.common.xacro" />
-    <xacro:include filename="$(find plato_description)/urdf/xacro/optimo.xacro" />
-    <xacro:include filename="$(find plato_description)/urdf/xacro/aristo_description.xacro" />
-    <xacro:include filename="$(find plato_description)/urdf/ros2_control/optimo.ros2_control.xacro" />
-    <xacro:include filename="$(find plato_description)/urdf/ros2_control/plato_mujoco.xacro" />
-    <mujoco>
-      <compiler meshdir="meshes/"/>
-    </mujoco>
-    <link name="world"/>
-    <!-- Add the arm, optional hand, and ros2_control -->
-    <xacro:optimo
-      prefix="$(arg prefix)"/>
-    <xacro:if value="$(arg use_aristo_hand)">
-      <xacro:aristo_description
-        prefix="aristo_" />
-      <joint name="aristo_connector_to_hand_mount" type="fixed">
-        <origin xyz="0 0 0.01" rpy="0 -1.57 3.1416"/>
-        <parent link="end_effector"/>
-        <child link="aristo_hand_mount"/>
-      </joint>
-    </xacro:if>
-    <!-- MuJoCo sim: unified ros2_control with all 15 joints -->
-    <xacro:if value="$(arg use_mujoco_sim)">
-      <ros2_control name="MujocoSystem" type="system">
-        <xacro:plato_mujoco_hardware
-            mujoco_model="$(arg mujoco_model)"
-            headless="$(arg headless)" />
-        <!-- Arm joints (7-DOF) -->
-        <joint name="joint1">
-            <command_interface name="position" />
-            <command_interface name="velocity" />
-            <command_interface name="effort">
-                <param name="min">-79</param>
-                <param name="max">79</param>
-            </command_interface>
-            <state_interface name="position" />
-            <state_interface name="velocity" />
-            <state_interface name="effort" />
-        </joint>
-        <joint name="joint2">
-            <command_interface name="position" />
-            <command_interface name="velocity" />
-            <command_interface name="effort">
-                <param name="min">-95</param>
-                <param name="max">95</param>
-            </command_interface>
-            <state_interface name="position" />
-            <state_interface name="velocity" />
-            <state_interface name="effort" />
-        </joint>
-        <joint name="joint3">
-            <command_interface name="position" />
-            <command_interface name="velocity" />
-            <command_interface name="effort">
-                <param name="min">-32</param>
-                <param name="max">32</param>
-            </command_interface>
-            <state_interface name="position" />
-            <state_interface name="velocity" />
-            <state_interface name="effort" />
-        </joint>
-        <joint name="joint4">
-            <command_interface name="position" />
-            <command_interface name="velocity" />
-            <command_interface name="effort">
-                <param name="min">-40</param>
-                <param name="max">40</param>
-            </command_interface>
-            <state_interface name="position" />
-            <state_interface name="velocity" />
-            <state_interface name="effort" />
-        </joint>
-        <joint name="joint5">
-            <command_interface name="position" />
-            <command_interface name="velocity" />
-            <command_interface name="effort">
-                <param name="min">-15</param>
-                <param name="max">15</param>
-            </command_interface>
-            <state_interface name="position" />
-            <state_interface name="velocity" />
-            <state_interface name="effort" />
-        </joint>
-        <joint name="joint6">
-            <command_interface name="position" />
-            <command_interface name="velocity" />
-            <command_interface name="effort">
-                <param name="min">-15</param>
-                <param name="max">15</param>
-            </command_interface>
-            <state_interface name="position" />
-            <state_interface name="velocity" />
-            <state_interface name="effort" />
-        </joint>
-        <joint name="joint7">
-            <command_interface name="position" />
-            <command_interface name="velocity" />
-            <command_interface name="effort">
-                <param name="min">-15</param>
-                <param name="max">15</param>
-            </command_interface>
-            <state_interface name="position" />
-            <state_interface name="velocity" />
-            <state_interface name="effort" />
-        </joint>
-        <!-- Hand joints (8-DOF) -->
-        <joint name="aristo_joint1">
-            <command_interface name="position" />
-            <command_interface name="velocity" />
-            <command_interface name="effort">
-                <param name="min">-10</param>
-                <param name="max">10</param>
-            </command_interface>
-            <state_interface name="position" />
-            <state_interface name="velocity" />
-            <state_interface name="effort" />
-        </joint>
-        <joint name="aristo_joint2">
-            <command_interface name="position" />
-            <command_interface name="velocity" />
-            <command_interface name="effort">
-                <param name="min">-10</param>
-                <param name="max">10</param>
-            </command_interface>
-            <state_interface name="position" />
-            <state_interface name="velocity" />
-            <state_interface name="effort" />
-        </joint>
-        <joint name="aristo_joint3">
-            <command_interface name="position" />
-            <command_interface name="velocity" />
-            <command_interface name="effort">
-                <param name="min">-10</param>
-                <param name="max">10</param>
-            </command_interface>
-            <state_interface name="position" />
-            <state_interface name="velocity" />
-            <state_interface name="effort" />
-        </joint>
-        <joint name="aristo_joint4">
-            <command_interface name="position" />
-            <command_interface name="velocity" />
-            <command_interface name="effort">
-                <param name="min">-10</param>
-                <param name="max">10</param>
-            </command_interface>
-            <state_interface name="position" />
-            <state_interface name="velocity" />
-            <state_interface name="effort" />
-        </joint>
-        <joint name="aristo_joint5">
-            <command_interface name="position" />
-            <command_interface name="velocity" />
-            <command_interface name="effort">
-                <param name="min">-10</param>
-                <param name="max">10</param>
-            </command_interface>
-            <state_interface name="position" />
-            <state_interface name="velocity" />
-            <state_interface name="effort" />
-        </joint>
-        <joint name="aristo_joint6">
-            <command_interface name="position" />
-            <command_interface name="velocity" />
-            <command_interface name="effort">
-                <param name="min">-10</param>
-                <param name="max">10</param>
-            </command_interface>
-            <state_interface name="position" />
-            <state_interface name="velocity" />
-            <state_interface name="effort" />
-        </joint>
-        <joint name="aristo_joint7">
-            <command_interface name="position" />
-            <command_interface name="velocity" />
-            <command_interface name="effort">
-                <param name="min">-10</param>
-                <param name="max">10</param>
-            </command_interface>
-            <state_interface name="position" />
-            <state_interface name="velocity" />
-            <state_interface name="effort" />
-        </joint>
-        <joint name="aristo_joint8">
-            <command_interface name="position" />
-            <command_interface name="velocity" />
-            <command_interface name="effort">
-                <param name="min">-10</param>
-                <param name="max">10</param>
-            </command_interface>
-            <state_interface name="position" />
-            <state_interface name="velocity" />
-            <state_interface name="effort" />
-        </joint>
-      </ros2_control>
-    </xacro:if>
-    <!-- Non-MuJoCo: use original Ignition/hardware ros2_control (arm only) -->
-    <xacro:unless value="$(arg use_mujoco_sim)">
-      <xacro:optimo_ros2_control use_sim_hardware="$(arg use_sim_hardware)" prefix="$(arg prefix)" robot_index="$(arg robot_index)" ns="$(arg ns)" />
-    </xacro:unless>
+<robot name="plato_hand" xmlns:xacro="http://www.ros.org/wiki/xacro">
+  <xacro:arg name="fake_hardware" default="false"/>
+  <xacro:arg name="zeroing" default="false"/>
+  <xacro:include filename="$(find plato_description)/urdf/xacro/plato_description.xacro"/>
+  <xacro:include filename="$(find plato_description)/urdf/ros2_control/plato.ros2_control.xacro"/>
+  <xacro:plato_description connector_link="world" xyz="0 0 0" rpy="0 0 0"/>
+  <xacro:plato_ros2_control
+    name="plato_ros2_control"
+    fake_hardware="$(arg fake_hardware)"
+    zeroing="$(arg zeroing)"/>
 </robot>

File: description/plato_description/urdf/ros2_control/aristo.ros2_control.xacro (robot description, xacro)
@@ -1,5 +1,5 @@
 <?xml version="0.06.0"?>
 <robot xmlns:xacro="http://www.ros.org/wiki/xacro">
-    <xacro:macro name="aristo_ros2_control" params="name fake_hardware='false'">
+    <xacro:macro name="aristo_ros2_control" params="name fake_hardware='false' zeroing='false' actuator_config_yaml_path=''">
         <!-- Normalize fake_hardware values so callers can pass true/False, 1/0, or strings -->
         <xacro:property name="use_mock" value="${fake_hardware == 'true' or fake_hardware == 'True' or fake_hardware == '1' or fake_hardware == 1 or fake_hardware == True}"/>
@@ -12,5 +12,9 @@
                 </xacro:if>
                 <xacro:unless value="${use_mock}">
-                    <plugin>plato2_hardware_interface/PLATO2Hardware</plugin>
+                    <plugin>aristo_hardware_interface/AristoHardware</plugin>
+                    <param name="zeroing">${zeroing}</param>
+                    <xacro:if value="${actuator_config_yaml_path != ''}">
+                        <param name="actuator_config_yaml_path">${actuator_config_yaml_path}</param>
+                    </xacro:if>
                 </xacro:unless>
             </hardware>
