Commit message: wip

File: description/plato_description/urdf/xacro/aristo_description.xacro (robot description, xacro)
@@ -2,20 +2,26 @@
 <robot xmlns:xacro="http://www.ros.org/wiki/xacro">
   <!--
-    Macro: builds the hand geometry/tree rooted at `${prefix}hand_mount`.
+    Macro: builds the hand and attaches it to `connector_link` with a fixed joint.
     Usage:
-      <xacro:aristo_description/>
+      <xacro:aristo_description connector_link="world" xyz="0 0 0" rpy="0 0 0"/>
   -->
-  <xacro:macro name="aristo_description" params="prefix:='aristo_'">
+  <xacro:macro name="aristo_description" params="connector_link xyz:='0 0 0' rpy:='0 0 0'">
     <!-- Create hand_mount link as intermediate frame -->
-    <link name="${prefix}hand_mount">
-    </link>
+    <link name="hand_mount">
+    </link>
+    <!-- Attach hand_mount to the provided connector link -->
+    <joint name="connector_to_hand_mount" type="fixed">
+      <origin xyz="0 0 0" rpy="0 0 0"/>
+      <parent link="${connector_link}"/>
+      <child link="hand_mount"/>
+    </joint>
     <!-- Rotate hand_base 90 degrees around Z to point in +X direction -->
-    <joint name="${prefix}hand_mount_to_base" type="fixed">
+    <joint name="hand_mount_to_base" type="fixed">
       <origin xyz="0 0 0" rpy="0 0 1.5708"/>
-      <parent link="${prefix}hand_mount"/>
-      <child link="${prefix}hand_base"/>
+      <parent link="hand_mount"/>
+      <child link="hand_base"/>
     </joint>
     <!-- Base link of the hand -->
-    <link name="${prefix}hand_base">
+    <link name="hand_base">
       <inertial>
         <origin xyz="1.14624e-05 -0.0735402 0.00270001" rpy="0 0 0"/>
@@ -26,5 +32,5 @@
         <origin xyz="1.14624e-05 -0.0735402 0.00270001" rpy="0 0 0"/>
         <geometry>
-          <mesh filename="package://plato_description/urdf/meshes/hand_base.stl"/>
+          <mesh filename="package://plato_description/meshes/hand_base.stl"/>
         </geometry>
         <material name="hand_base_parts_material">
@@ -35,27 +41,27 @@
         <origin xyz="1.14624e-05 -0.0735402 0.00270001" rpy="0 0 0"/>
         <geometry>
-          <mesh filename="package://plato_description/urdf/meshes/col_hand_base.stl"/>
+          <mesh filename="package://plato_description/meshes/hand_base.stl"/>
         </geometry>
       </collision>
     </link>
     <!-- thumb_distal_tactile: tactile sensor frame 4.73 cm distal of thumb_distal -->
-    <link name="${prefix}thumb_distal_tactile" />
-    <joint name="${prefix}thumb_distal_to_tactile" type="fixed">
+    <link name="thumb_distal_tactile" />
+    <joint name="thumb_distal_to_tactile" type="fixed">
       <!-- translate 0.0473 m (4.73 cm) along the distal link local +x -->
   <!-- orient tactile frame so Z+ points downward while keeping +X forward: rotate pi around X -->
   <!-- keep thumb translation, mirror orientation of index (invert yaw) -->
   <origin xyz="-0.0523 0.01 -0.0025" rpy="0 1.57 1.57"/>
-      <parent link="${prefix}thumb_distal"/>
-      <child link="${prefix}thumb_distal_tactile"/>
+      <parent link="thumb_distal"/>
+      <child link="thumb_distal_tactile"/>
     </joint>
     <!-- thumb_fingertip: fingertip frame at the end of thumb -->
-    <link name="${prefix}thumb_fingertip" />
-    <joint name="${prefix}thumb_distal_to_fingertip" type="fixed">
+    <link name="thumb_fingertip" />
+    <joint name="thumb_distal_to_fingertip" type="fixed">
       <origin xyz="-0.066 0 0" rpy="0 0 0"/>
-      <parent link="${prefix}thumb_distal"/>
-      <child link="${prefix}thumb_fingertip"/>
+      <parent link="thumb_distal"/>
+      <child link="thumb_fingertip"/>
     </joint>
     <!-- thumb_metacarpal -->
-    <link name="${prefix}thumb_metacarpal">
+    <link name="thumb_metacarpal">
       <inertial>
         <origin xyz="5.08388e-05 -0.0186588 0.0228524" rpy="0 0 0"/>
@@ -66,5 +72,5 @@
         <origin xyz="5.08388e-05 -0.0186588 0.0228524" rpy="-1.5708 0 -2.97318e-15"/>
         <geometry>
-          <mesh filename="package://plato_description/urdf/meshes/thumb_metacarpal.stl"/>
+          <mesh filename="package://plato_description/meshes/thumb_metacarpal.stl"/>
         </geometry>
         <material name="thumb_metacarpal_parts_material">
@@ -75,10 +81,10 @@
         <origin xyz="5.08388e-05 -0.0186588 0.0228524" rpy="-1.5708 0 -2.97318e-15"/>
         <geometry>
-          <mesh filename="package://plato_description/urdf/meshes/col_thumb_metacarpal.stl"/>
+          <mesh filename="package://plato_description/meshes/thumb_metacarpal.stl"/>
         </geometry>
       </collision>
     </link>
     <!-- thumb_actuators -->
-    <link name="${prefix}thumb_actuators">
+    <link name="thumb_actuators">
       <inertial>
         <origin xyz="0.00119788 -0.0189545 -0.0225138" rpy="0 0 0"/>
@@ -89,5 +95,5 @@
         <origin xyz="0.00119788 -0.0189545 -0.0225138" rpy="0 0 -1.5708"/>
         <geometry>
-          <mesh filename="package://plato_description/urdf/meshes/thumb_actuators.stl"/>
+          <mesh filename="package://plato_description/meshes/thumb_actuators.stl"/>
         </geometry>
         <material name="thumb_actuators_parts_material">
@@ -98,10 +104,10 @@
         <origin xyz="0.00119788 -0.0189545 -0.0225138" rpy="0 0 -1.5708"/>
         <geometry>
-          <mesh filename="package://plato_description/urdf/meshes/col_thumb_actuators.stl"/>
+          <mesh filename="package://plato_description/meshes/thumb_actuators.stl"/>
         </geometry>
       </collision>
     </link>
     <!-- thumb_proximal -->
-    <link name="${prefix}thumb_proximal">
+    <link name="thumb_proximal">
       <inertial>
         <origin xyz="0.0275353 8.61887e-05 0.00673205" rpy="0 0 0"/>
@@ -112,5 +118,5 @@
         <origin xyz="0.0275353 8.61887e-05 0.00673205" rpy="1.5708 -1.5708 0"/>
         <geometry>
-          <mesh filename="package://plato_description/urdf/meshes/thumb_proximal.stl"/>
+          <mesh filename="package://plato_description/meshes/thumb_proximal.stl"/>
         </geometry>
         <material name="thumb_proximal_parts_material">
@@ -121,10 +127,10 @@
         <origin xyz="0.0275353 8.61887e-05 0.00673205" rpy="1.5708 -1.5708 0"/>
         <geometry>
-          <mesh filename="package://plato_description/urdf/meshes/col_thumb_proximal.stl"/>
+          <mesh filename="package://plato_description/meshes/thumb_proximal.stl"/>
         </geometry>
       </collision>
     </link>
     <!-- thumb_distal -->
-    <link name="${prefix}thumb_distal">
+    <link name="thumb_distal">
       <inertial>
         <origin xyz="-0.0330685 -0.00101822 -0.00300906" rpy="0 0 0"/>
@@ -135,5 +141,5 @@
         <origin xyz="-0.0330685 -0.00101822 -0.00300906" rpy="-1.5708 -1.5708 0"/>
         <geometry>
-          <mesh filename="package://plato_description/urdf/meshes/thumb_distal.stl"/>
+          <mesh filename="package://plato_description/meshes/thumb_distal.stl"/>
         </geometry>
         <material name="thumb_distal_parts_material">
@@ -144,39 +150,39 @@
         <origin xyz="-0.0330685 -0.00101822 -0.00300906" rpy="-1.5708 -1.5708 0"/>
         <geometry>
-          <mesh filename="package://plato_description/urdf/meshes/col_thumb_distal.stl"/>
+          <mesh filename="package://plato_description/meshes/thumb_distal.stl"/>
         </geometry>
       </collision>
     </link>
     <!-- Thumb joints -->
-    <joint name="${prefix}joint1" type="revolute">
+    <joint name="joint1" type="revolute">
       <origin xyz="4.56293e-16 -0.044 -0.0285" rpy="1.5708 0 0"/>
-      <parent link="${prefix}hand_base"/>
-      <child link="${prefix}thumb_metacarpal"/>
+      <parent link="hand_base"/>
+      <child link="thumb_metacarpal"/>
       <axis xyz="0 0 1"/>
       <limit effort="10" velocity="10" lower="-0.785398" upper="0.785398"/>
     </joint>
-    <joint name="${prefix}joint2" type="revolute">
+    <joint name="joint2" type="revolute">
       <origin xyz="-1.42383e-10 -0.0315 0.025" rpy="-1.5708 1.5708 0"/>
-      <parent link="${prefix}thumb_metacarpal"/>
-      <child link="${prefix}thumb_actuators"/>
+      <parent link="thumb_metacarpal"/>
+      <child link="thumb_actuators"/>
       <axis xyz="0 0 1"/>
       <limit effort="10" velocity="10" lower="-1.5708" upper="1.5708"/>
     </joint>
-    <joint name="${prefix}joint3" type="revolute">
+    <joint name="joint3" type="revolute">
       <origin xyz="-0.022 -0.0305 -0.0235" rpy="-1.5708 0 3.14159"/>
-      <parent link="${prefix}thumb_actuators"/>
-      <child link="${prefix}thumb_proximal"/>
+      <parent link="thumb_actuators"/>
+      <child link="thumb_proximal"/>
       <axis xyz="0 0 1"/>
       <limit effort="10" velocity="10" lower="-1.0472" upper="1.0472"/>
     </joint>
-    <joint name="${prefix}joint4" type="revolute">
+    <joint name="joint4" type="revolute">
       <origin xyz="0.06 0 0.0105" rpy="0 0 3.14159"/>
-      <parent link="${prefix}thumb_proximal"/>
-      <child link="${prefix}thumb_distal"/>
+      <parent link="thumb_proximal"/>
+      <child link="thumb_distal"/>
       <axis xyz="0 0 1"/>
       <limit effort="10" velocity="10" lower="-2.0944" upper="1.0472"/>
     </joint>
     <!-- index_proximal -->
-    <link name="${prefix}index_proximal">
+    <link name="index_proximal">
       <inertial>
         <origin xyz="0.0275353 -8.61566e-05 0.00673211" rpy="0 0 0"/>
@@ -187,5 +193,5 @@
         <origin xyz="0.0275353 -8.61566e-05 0.00673211" rpy="1.5708 -1.5708 0"/>
         <geometry>
-          <mesh filename="package://plato_description/urdf/meshes/index_proximal.stl"/>
+          <mesh filename="package://plato_description/meshes/index_proximal.stl"/>
         </geometry>
         <material name="index_proximal_parts_material">
@@ -196,10 +202,10 @@
         <origin xyz="0.0275353 -8.61566e-05 0.00673211" rpy="1.5708 -1.5708 0"/>
         <geometry>
-          <mesh filename="package://plato_description/urdf/meshes/col_index_proximal.stl"/>
+          <mesh filename="package://plato_description/meshes/index_proximal.stl"/>
         </geometry>
       </collision>
     </link>
     <!-- index_distal -->
-    <link name="${prefix}index_distal">
+    <link name="index_distal">
       <inertial>
         <origin xyz="-0.0330685 0.00101822 -0.00299094" rpy="0 0 0"/>
@@ -210,5 +216,5 @@
         <origin xyz="-0.0330685 0.00101822 -0.00299094" rpy="-1.5708 -1.5708 0"/>
         <geometry>
-          <mesh filename="package://plato_description/urdf/meshes/index_distal.stl"/>
+          <mesh filename="package://plato_description/meshes/index_distal.stl"/>
         </geometry>
         <material name="index_distal_parts_material">
@@ -219,56 +225,56 @@
         <origin xyz="-0.0330685 0.00101822 -0.00299094" rpy="-1.5708 -1.5708 0"/>
         <geometry>
-          <mesh filename="package://plato_description/urdf/meshes/col_index_distal.stl"/>
+          <mesh filename="package://plato_description/meshes/index_distal.stl"/>
         </geometry>
       </collision>
     </link>
     <!-- Index joints -->
-    <joint name="${prefix}joint5" type="revolute">
+    <joint name="joint5" type="revolute">
       <origin xyz="0.0305 -0.113 0.0145" rpy="-1.5708 0 -1.5708"/>
-      <parent link="${prefix}hand_base"/>
-      <child link="${prefix}index_proximal"/>
+      <parent link="hand_base"/>
+      <child link="index_proximal"/>
       <axis xyz="0 0 1"/>
       <limit effort="10" velocity="10" lower="-1.0472" upper="1.0472"/>
     </joint>
-    <joint name="${prefix}joint6" type="revolute">
+    <joint name="joint6" type="revolute">
       <origin xyz="0.06 0 0.0105" rpy="0 0 3.14159"/>
-      <parent link="${prefix}index_proximal"/>
-      <child link="${prefix}index_distal"/>
+      <parent link="index_proximal"/>
+      <child link="index_distal"/>
       <axis xyz="0 0 1"/>
       <limit effort="10" velocity="10" lower="-1.0472" upper="2.0944"/>
     </joint>
     <!-- index_distal_tactile: tactile sensor frame 4.73 cm distal of index_distal -->
-    <link name="${prefix}index_distal_tactile" />
-    <joint name="${prefix}index_distal_to_tactile" type="fixed">
+    <link name="index_distal_tactile" />
+    <joint name="index_distal_to_tactile" type="fixed">
       <!-- translate 0.0473 m (4.73 cm) along the distal link local +x -->
   <!-- orient tactile frame so Z+ points downward while keeping +X forward: rotate pi around X -->
   <origin xyz="-0.0523 -0.01 -0.0025" rpy="0 -1.57 1.57"/>
-      <parent link="${prefix}index_distal"/>
-      <child link="${prefix}index_distal_tactile"/>
+      <parent link="index_distal"/>
+      <child link="index_distal_tactile"/>
     </joint>
     <!-- index_fingertip: fingertip frame at the end of index finger -->
-    <link name="${prefix}index_fingertip" />
-    <joint name="${prefix}index_distal_to_fingertip" type="fixed">
+    <link name="index_fingertip" />
+    <joint name="index_distal_to_fingertip" type="fixed">
       <origin xyz="-0.066 0 0" rpy="0 0 0"/>
-      <parent link="${prefix}index_distal"/>
-      <child link="${prefix}index_fingertip"/>
+      <parent link="index_distal"/>
+      <child link="index_fingertip"/>
     </joint>
       <!-- Middle joints -->
-    <joint name="${prefix}joint7" type="revolute">
+    <joint name="joint7" type="revolute">
       <origin xyz="-0.0305 -0.113 0.0145" rpy="-1.5708 0 -1.5708"/>
-      <parent link="${prefix}hand_base"/>
-      <child link="${prefix}middle_proximal"/>
+      <parent link="hand_base"/>
+      <child link="middle_proximal"/>
       <axis xyz="0 0 1"/>
       <limit effort="10" velocity="10" lower="-1.0472" upper="1.0472"/>
     </joint>
-    <joint name="${prefix}joint8" type="revolute">
+    <joint name="joint8" type="revolute">
       <origin xyz="0.06 0 -0.0105" rpy="0 0 -3.14159"/>
-      <parent link="${prefix}middle_proximal"/>
-      <child link="${prefix}middle_distal"/>
+      <parent link="middle_proximal"/>
+      <child link="middle_distal"/>
       <axis xyz="0 0 1"/>
       <limit effort="10" velocity="10" lower="-1.0472" upper="2.0944"/>
     </joint>
     <!-- middle_proximal -->
-    <link name="${prefix}middle_proximal">
+    <link name="middle_proximal">
       <inertial>
         <origin xyz="0.0275353 -8.61887e-05 -0.00673205" rpy="0 0 0"/>
@@ -279,5 +285,5 @@
         <origin xyz="0.0275353 -8.61887e-05 -0.00673205" rpy="1.5708 -1.5708 0"/>
         <geometry>
-          <mesh filename="package://plato_description/urdf/meshes/middle_proximal.stl"/>
+          <mesh filename="package://plato_description/meshes/middle_proximal.stl"/>
         </geometry>
         <material name="middle_proximal_parts_material">
@@ -288,10 +294,10 @@
         <origin xyz="0.0275353 -8.61887e-05 -0.00673205" rpy="1.5708 -1.5708 0"/>
         <geometry>
-          <mesh filename="package://plato_description/urdf/meshes/col_middle_proximal.stl"/>
+          <mesh filename="package://plato_description/meshes/middle_proximal.stl"/>
         </geometry>
       </collision>
     </link>
     <!-- middle_distal -->
-    <link name="${prefix}middle_distal">
+    <link name="middle_distal">
       <inertial>
         <origin xyz="-0.0330685 0.00101822 0.00300906" rpy="0 0 0"/>
@@ -302,5 +308,5 @@
         <origin xyz="-0.0330685 0.00101822 0.00300906" rpy="-1.5708 -1.5708 0"/>
         <geometry>
-          <mesh filename="package://plato_description/urdf/meshes/middle_distal.stl"/>
+          <mesh filename="package://plato_description/meshes/middle_distal.stl"/>
         </geometry>
         <material name="middle_distal_parts_material">
@@ -311,23 +317,23 @@
         <origin xyz="-0.0330685 0.00101822 0.00300906" rpy="-1.5708 -1.5708 0"/>
         <geometry>
-          <mesh filename="package://plato_description/urdf/meshes/col_middle_distal.stl"/>
+          <mesh filename="package://plato_description/meshes/middle_distal.stl"/>
         </geometry>
       </collision>
     </link>
     <!-- middle_distal_tactile: tactile sensor frame 4.73 cm distal of middle_distal -->
-    <link name="${prefix}middle_distal_tactile" />
-    <joint name="${prefix}middle_distal_to_tactile" type="fixed">
+    <link name="middle_distal_tactile" />
+    <joint name="middle_distal_to_tactile" type="fixed">
       <!-- translate 0.0473 m (4.73 cm) along the distal link local +x -->
   <!-- orient tactile frame so Z+ points downward while keeping +X forward: rotate pi around X -->
   <origin xyz="-0.0523 -0.01 -0.0025" rpy="0 -1.57 1.57"/>
-      <parent link="${prefix}middle_distal"/>
-      <child link="${prefix}middle_distal_tactile"/>
+      <parent link="middle_distal"/>
+      <child link="middle_distal_tactile"/>
     </joint>
     <!-- middle_fingertip: fingertip frame at the end of middle finger -->
-    <link name="${prefix}middle_fingertip" />
-    <joint name="${prefix}middle_distal_to_fingertip" type="fixed">
+    <link name="middle_fingertip" />
+    <joint name="middle_distal_to_fingertip" type="fixed">
       <origin xyz="-0.066 0 0" rpy="0 0 0"/>
-      <parent link="${prefix}middle_distal"/>
-      <child link="${prefix}middle_fingertip"/>
+      <parent link="middle_distal"/>
+      <child link="middle_fingertip"/>
     </joint>
   </xacro:macro>
